File: hardware/AmiWiFi.kicad_sch (KiCad schematic)
At the start: 56 parts, among them J1 TYPE-C 6P, J2 DB25 MALE / MAS original, U1 LD2981ABU33TR, U2 SN74LVC4245APWR, U3 SN74LVC125APWR, U4 SN74LVC4245APWR, U5 SN74LVC1G10DBVR, U6 SN74LVC1G10DBVR, U7 Raspberry Pi Pico 2 W, U8 SN74LVC2G07DCKR

Commit message: Align KiCad footprints with user hardware revision and add missing LED components
Parts:
- added D2: LED, AmiWiFi:LED_0603_HandSolder_D2, symbol AmiWiFi:LED_D2
- added R18: 330, AmiWiFi:R0402_R18, symbol AmiWiFi:Part_R10
Connections:
- net +3V3_IF: now also R18.1
- net GND: now also D2.1 (K)
- new net: D2.2 (A), R18.2
